File: hardware/PowerDistributionBoard-V2.0/staff-pdb-a.brd (EAGLE design)
At the start: 20.3 x 21.6 mm, 4 parts, among them J3 B4B-XH-A(LF)(SN)

Commit message: rearranging files
Connections:
- net A renamed GND
- net B renamed S1
- net C renamed S2
- net D renamed VCC
Routing:
- net VCC: track 25.4 -> 29.6 mm, vias 0 -> 1
Other:
- board size 20.3 x 21.6 mm -> 21.6 x 21.6 mm
- board text added: "+"
- board text added: "-"
- board text added: "1"
- board text added: "2"
- board text added: "PDB - A"
- board text removed: "A"
- board text removed: "B"
- board text removed: "C"
- board text removed: "D"
