File: hardware/PowerDistributionBoard-V2.0/staff-pdb-a.sch (EAGLE design)
At the start: 4 parts, among them J3 B4B-XH-A(LF)(SN)

Commit message: rearranging files
Connections:
- net A renamed GND
- net B renamed S1
- net C renamed S2
- net D renamed VCC
Changed lines of the file:
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@@
 <?xml version="1.0" encoding="utf-8"?>
 <!DOCTYPE eagle SYSTEM "eagle.dtd">
-<eagle version="9.2.2">
+<eagle version="9.6.2">
 <drawing>
 <settings>
-<setting alwaysvectorfont="yes"/>
+<setting alwaysvectorfont="no"/>
 <setting verticaltext="up"/>
 </settings>
@@
 </busses>
 <nets>
-<net name="A" class="0">
+<net name="GND" class="0">
 <segment>
 <pinref part="J2" gate="G$1" pin="1"/>
@@
 </segment>
 </net>
-<net name="B" class="0">
+<net name="S1" class="0">
 <segment>
 <pinref part="J2" gate="G$1" pin="2"/>
@@
 </segment>
 </net>
-<net name="C" class="0">
+<net name="S2" class="0">
 <segment>
 <pinref part="J2" gate="G$1" pin="3"/>
@@
 </segment>
 </net>
-<net name="D" class="0">
+<net name="VCC" class="0">
 <segment>
 <pinref part="J2" gate="G$1" pin="4"/>
