File: hardware/PowerDistributionBoard-V2.0/staff-pdb-b.brd (EAGLE design)
At the start: 21.6 x 21.6 mm, 5 parts, among them J3 B5B-XH-A(LF)(SN)

Commit message: rearranging files
Parts:
- removed D1: BAT60J, diode:SOD323_ST
- J3: value B5B-XH-A(LF)(SN) -> B4B-XH-A(LF)(SN); device B4B-XH-A_LF__SN_:JST_B5B-XH-A(LF)(SN) -> RoverWing-V1.5:JST_B4B-XH-A(LF)(SN)
- moved J3 5.39 mm to (0.00, -3.81), turned to 90 degrees
Connections:
- net A renamed S2
- removed net B: J1.2, J2.2, J3.4, J4.2
- removed net VCC-MCU: D1.C, J3.1, J4.4
- new net S1: J1.2, J2.2, J3.2, J4.2
- net GND: now also J1.4, J2.4, J3.4, J4.4; no longer J1.1, J2.1, J3.5, J4.1
- net VCC: now also J1.1, J2.1, J3.1, J4.1; no longer D1.A, J1.4, J2.4, J3.2
Routing:
- net S1: track 0.00 -> 31.7 mm
- net B: track 30.3 -> 0.00 mm
- net VCC: track 19.8 -> 30.0 mm, vias 0 -> 1
- net S2: track 33.6 -> 25.1 mm, vias 1 -> 0
- net VCC-MCU: track 7.78 -> 0.00 mm
- net GND: track 29.3 -> 25.3 mm
Other:
- outline, holes or cut-outs redrawn
- board text added: "-"
- board text added: "1"
- board text added: "2"
- board text added: "PDB - B"
- board text removed: "A"
- board text removed: "B"
- board text removed: "G"
